Commit message: 添加了一些存活检测保护

File: src/control_launch/urdf/robot.urdf (robot description, URDF)
Before this commit: robot chassis, 5 links, 4 joints
Links:
- added link front_left_leg
- added link front_right_leg
- added link rear_left_leg
- added link rear_right_leg
Joints:
- added joint front_left_leg_joint: type revolute, parent base_link, child front_left_leg, origin xyz=0.2 0.15 0 rpy=0 0 0, axis 0 1 0, limit lower=-1.57 upper=1.57 effort=10.0 velocity=10.0
- added joint front_right_leg_joint: type revolute, parent base_link, child front_right_leg, origin xyz=0.2 -0.15 0 rpy=0 0 0, axis 0 1 0, limit lower=-1.57 upper=1.57 effort=10.0 velocity=10.0
- added joint rear_left_leg_joint: type revolute, parent base_link, child rear_left_leg, origin xyz=-0.2 0.15 0 rpy=0 0 0, axis 0 1 0, limit lower=-1.57 upper=1.57 effort=10.0 velocity=10.0
- added joint rear_right_leg_joint: type revolute, parent base_link, child rear_right_leg, origin xyz=-0.2 -0.15 0 rpy=0 0 0, axis 0 1 0, limit lower=-1.57 upper=1.57 effort=10.0 velocity=10.0
