Commit message: 上位机leg控制完成版

File: src/robot/urdf/robot.urdf (robot description, URDF)
Before this commit: robot robot, 9 links, 8 joints
Joints:
- joint front_left_leg_joint: axis 0 1 0 -> (none); limit lower=-1.57 upper=1.57 effort=10.0 velocity=10.0 -> (none); origin xyz=0.2 0.15 0 rpy=0 0 0 -> (none); type revolute -> fixed
- joint front_right_leg_joint: axis 0 1 0 -> (none); limit lower=-1.57 upper=1.57 effort=10.0 velocity=10.0 -> (none); origin xyz=0.2 -0.15 0 rpy=0 0 0 -> (none); type revolute -> fixed
- joint rear_left_leg_joint: axis 0 1 0 -> (none); limit lower=-1.57 upper=1.57 effort=10.0 velocity=10.0 -> (none); origin xyz=-0.2 0.15 0 rpy=0 0 0 -> (none); type revolute -> fixed
- joint rear_right_leg_joint: axis 0 1 0 -> (none); limit lower=-1.57 upper=1.57 effort=10.0 velocity=10.0 -> (none); origin xyz=-0.2 -0.15 0 rpy=0 0 0 -> (none); type revolute -> fixed

Commit message: 删除仲裁部分，遥控器准备移交导航端，提供麦轮里程计接收demo

File: src/robot/urdf/robot.urdf (robot description, URDF)
Before this commit: robot robot, 9 links, 8 joints
Joints:
- joint front_left_wheel_joint: origin xyz=0.2 0.15 -0.05 rpy=0 0 0 -> xyz=0.27362 0.213 -0.05 rpy=0 0 0
- joint front_right_wheel_joint: origin xyz=0.2 -0.15 -0.05 rpy=0 0 0 -> xyz=0.27362 -0.213 -0.05 rpy=0 0 0
- joint rear_left_wheel_joint: origin xyz=-0.2 0.15 -0.05 rpy=0 0 0 -> xyz=-0.27362 0.213 -0.05 rpy=0 0 0
- joint rear_right_wheel_joint: origin xyz=-0.2 -0.15 -0.05 rpy=0 0 0 -> xyz=-0.27362 -0.213 -0.05 rpy=0 0 0
